File: pcb/LifterV03.brd (EAGLE design)
At the start: 109.2 x 25 mm, 60 parts, among them IC2 TL072D

Commit message: BigMac changes.
Parts:
- turned C10 to 180 degrees
- turned C12 to 180 degrees
- turned R12 to 0 degrees
Connections:
- removed net N$39 (its old number): OPAMP_RO.8, R26.2, R6.2
- new net N$41: C12.1, OPAMP_RO.8, R26.2, R6.2
- net N$18: now also R12.1; no longer C10.2
- net N$23: now also C10.2; no longer C10.1, R12.1
- net N$24: now also C10.1
- net N$37: now also R26.1; no longer C12.2
- net N$38: now also C12.2; no longer C12.1, R26.1
Routing:
- net N$41: track 0.00 -> 21.8 mm
- net N$39 (its old number): track 16.7 -> 0.00 mm
- net N$37: track 81.1 -> 72.6 mm, vias 4 -> 1
- net N$23: track 87.2 -> 79.7 mm
- net N$38: track 86.4 -> 79.5 mm
- net N$18: track 82.6 -> 77.1 mm
- net N$24: track 16.9 -> 20.2 mm
- net N$39: track 41.6 -> 42.4 mm
- net VSS: track 112.1 -> 112.9 mm
- net N$3: track 40.5 -> 41.2 mm
- net N$28: track 50.5 -> 51.0 mm
Other:
- board text added: "mb'Lifter v03"
- board text removed: "mb'Lifter"
