File: pcb/LifterV03.sch (EAGLE design)
At the start: 60 parts, among them IC2 TL072D

Commit message: BigMac changes.
Connections:
- removed net N$39 (its old number): OPAMP_ROC.OUT, R26.2, R6.2
- new net N$41: C12.1, OPAMP_ROC.OUT, R26.2, R6.2
- net N$18: now also R12.1; no longer C10.2
- net N$23: now also C10.2; no longer C10.1, R12.1
- net N$24: now also C10.1
- net N$37: now also R26.1; no longer C12.2
- net N$38: now also C12.2; no longer C12.1, R26.1
Other:
- moved on the sheet: C10, C12, C9
